File: Schematics/CPU/CPU.kicad_pcb (KiCad board)
At the start: 2 copper layers, 109.2 x 106.7 mm, 69 parts, among them J1 3x32, J2 2x08, J3 2x08, J4 2x08, J5 2x01, J6 2x03, Q1 Q_NMOS_DGS, Q2 Q_NMOS_DGS, SW1 SW_DIP_x08, U1 68000D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

Commit message: a
Connections:
- U7 pad 1: /IS5 -> /IS4
- U7 pad 11: /IS4 -> /IS1
- U7 pad 12: /IS1 -> /IS2
- U7 pad 13: /IS2 -> /IS3
- U7 pad 2: /IS6 -> /IS5
- U7 pad 3: /IS3 -> /IS6
Routing:
- net /IS7: track 37.7 -> 3.46 mm
- net /IS6: track 35.7 -> 5.74 mm
- net /IS3: track 34.2 -> 5.08 mm, vias 2 -> 1
- net /IS5: track 32.2 -> 7.27 mm
- net /IS1: track 25.6 -> 4.73 mm
- net /IS4: track 27.1 -> 6.76 mm
- net /IS2: track 18.0 -> 4.57 mm, vias 0 -> 1
Changed lines of the file:
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@@
     (fp_line (start 9.74 5.01) (end -9.74 5.01) (layer "F.CrtYd") (width 0.05))
     (pad "1" thru_hole oval locked (at -8.89 3.76 180) (size 1.2 2) (drill 0.8) (layers *.Cu *.Mask)
-      (net 162 "/IS5") (pinfunction "I4") (pintype "input"))
+      (net 159 "/IS4") (pinfunction "I4") (pintype "input"))
     (pad "2" thru_hole oval locked (at -6.35 3.76 180) (size 1.2 2) (drill 0.8) (layers *.Cu *.Mask)
-      (net 160 "/IS6") (pinfunction "I5") (pintype "input"))
+      (net 162 "/IS5") (pinfunction "I5") (pintype "input"))
     (pad "3" thru_hole oval locked (at -3.81 3.76 180) (size 1.2 2) (drill 0.8) (layers *.Cu *.Mask)
-      (net 158 "/IS3") (pinfunction "I6") (pintype "input"))
+      (net 160 "/IS6") (pinfunction "I6") (pintype "input"))
     (pad "4" thru_hole oval locked (at -1.27 3.76 180) (size 1.2 2) (drill 0.8) (layers *.Cu *.Mask)
       (net 157 "/IS7") (pinfunction "I7") (pintype "input"))
@@
       (net 16 "GND") (pinfunction "IO") (pintype "input"))
     (pad "11" thru_hole oval locked (at 3.81 -3.76 180) (size 1.2 2) (drill 0.8) (layers *.Cu *.Mask)
-      (net 159 "/IS4") (pinfunction "I1") (pintype "input"))
+      (net 161 "/IS1") (pinfunction "I1") (pintype "input"))
     (pad "12" thru_hole oval locked (at 1.27 -3.76 180) (size 1.2 2) (drill 0.8) (layers *.Cu *.Mask)
-      (net 161 "/IS1") (pinfunction "I2") (pintype "input"))
+      (net 163 "/IS2") (pinfunction "I2") (pintype "input"))
     (pad "13" thru_hole oval locked (at -1.27 -3.76 180) (size 1.2 2) (drill 0.8) (layers *.Cu *.Mask)
-      (net 163 "/IS2") (pinfunction "I3") (pintype "input"))
+      (net 158 "/IS3") (pinfunction "I3") (pintype "input"))
     (pad "14" thru_hole oval locked (at -3.81 -3.76 180) (size 1.2 2) (drill 0.8) (layers *.Cu *.Mask)
       (net 133 "unconnected-(U7-Pad14)") (pinfunction "GS") (pintype "output+no_connect"))
@@
   (segment (start 29.21 48.514) (end 29.21 26.67) (width 0.2) (layer "B.Cu") (net 156))
   (segment (start 31.75 60.91) (end 30.48 59.64) (width 0.2) (layer "B.Cu") (net 156))
-  (segment (start 26.67 55.118) (end 60.96 55.118) (width 0.2) (layer "F.Cu") (net 157))
   (via (at 60.96 55.118) (size 0.55) (drill 0.35) (layers "F.Cu" "B.Cu") (net 157))
   (via (at 26.67 55.118) (size 0.55) (drill 0.35) (layers "F.Cu" "B.Cu") (net 157))
   (segment (start 26.67 53.39) (end 26.67 55.118) (width 0.2) (layer "B.Cu") (net 157))
   (segment (start 60.96 55.118) (end 60.96 53.39) (width 0.2) (layer "B.Cu") (net 157))
-  (segment (start 63.5 55.88) (end 34.29 55.88) (width 0.2) (layer "F.Cu") (net 158))
-  (via (at 63.5 55.88) (size 0.55) (drill 0.35) (layers "F.Cu" "B.Cu") (net 158))
+  (segment (start 60.96 60.91) (end 59.132 62.738) (width 0.2) (layer "F.Cu") (net 158))
   (via (at 34.29 55.88) (size 0.55) (drill 0.35) (layers "F.Cu" "B.Cu") (net 158))
-  (segment (start 63.5 53.39) (end 63.5 55.88) (width 0.2) (layer "B.Cu") (net 158))
   (segment (start 34.29 55.88) (end 34.29 53.39) (width 0.2) (layer "B.Cu") (net 158))
-  (segment (start 34.29 58.166) (end 55.88 58.166) (width 0.2) (layer "F.Cu") (net 159))
-  (via (at 55.88 58.166) (size 0.55) (drill 0.35) (layers "F.Cu" "B.Cu") (net 159))
   (via (at 34.29 58.166) (size 0.55) (drill 0.35) (layers "F.Cu" "B.Cu") (net 159))
+  (via (at 68.58 57.404) (size 0.55) (drill 0.35) (layers "F.Cu" "B.Cu") (net 159))
   (segment (start 34.29 58.166) (end 34.29 60.91) (width 0.2) (layer "B.Cu") (net 159))
-  (segment (start 55.88 60.91) (end 55.88 58.166) (width 0.2) (layer "B.Cu") (net 159))
-  (segment (start 36.83 56.642) (end 66.04 56.642) (width 0.2) (layer "F.Cu") (net 160))
+  (segment (start 68.58 53.39) (end 68.58 57.404) (width 0.2) (layer "B.Cu") (net 159))
   (via (at 36.83 56.642) (size 0.55) (drill 0.35) (layers "F.Cu" "B.Cu") (net 160))
-  (via (at 66.04 56.642) (size 0.55) (drill 0.35) (layers "F.Cu" "B.Cu") (net 160))
-  (segment (start 66.04 56.642) (end 66.04 53.39) (width 0.2) (layer "B.Cu") (net 160))
+  (via (at 63.5 55.88) (size 0.55) (drill 0.35) (layers "F.Cu" "B.Cu") (net 160))
+  (segment (start 63.5 53.39) (end 63.5 55.88) (width 0.2) (layer "B.Cu") (net 160))
   (segment (start 36.83 53.39) (end 36.83 56.642) (width 0.2) (layer "B.Cu") (net 160))
-  (segment (start 36.83 58.928) (end 58.42 58.928) (width 0.2) (layer "F.Cu") (net 161))
-  (via (at 58.42 58.928) (size 0.55) (drill 0.35) (layers "F.Cu" "B.Cu") (net 161))
+  (via (at 55.88 58.166) (size 0.55) (drill 0.35) (layers "F.Cu" "B.Cu") (net 161))
   (via (at 36.83 58.928) (size 0.55) (drill 0.35) (layers "F.Cu" "B.Cu") (net 161))
   (segment (start 36.83 58.928) (end 36.83 60.91) (width 0.2) (layer "B.Cu") (net 161))
-  (segment (start 58.42 60.91) (end 58.42 58.928) (width 0.2) (layer "B.Cu") (net 161))
-  (segment (start 68.58 57.404) (end 44.45 57.404) (width 0.2) (layer "F.Cu") (net 162))
+  (segment (start 55.88 60.91) (end 55.88 58.166) (width 0.2) (layer "B.Cu") (net 161))
+  (via (at 66.04 56.642) (size 0.55) (drill 0.35) (layers "F.Cu" "B.Cu") (net 162))
   (via (at 44.45 57.404) (size 0.55) (drill 0.35) (layers "F.Cu" "B.Cu") (net 162))
-  (via (at 68.58 57.404) (size 0.55) (drill 0.35) (layers "F.Cu" "B.Cu") (net 162))
-  (segment (start 68.58 53.39) (end 68.58 57.404) (width 0.2) (layer "B.Cu") (net 162))
+  (segment (start 66.04 56.642) (end 66.04 53.39) (width 0.2) (layer "B.Cu") (net 162))
   (segment (start 44.45 53.39) (end 44.45 57.404) (width 0.2) (layer "B.Cu") (net 162))
   (segment (start 46.278 62.738) (end 44.45 60.91) (width 0.2) (layer "F.Cu") (net 163))
-  (segment (start 59.132 62.738) (end 46.278 62.738) (width 0.2) (layer "F.Cu") (net 163))
-  (segment (start 60.96 60.91) (end 59.132 62.738) (width 0.2) (layer "F.Cu") (net 163))
+  (via (at 58.42 58.928) (size 0.55) (drill 0.35) (layers "F.Cu" "B.Cu") (net 163))
+  (segment (start 58.42 60.91) (end 58.42 58.928) (width 0.2) (layer "B.Cu") (net 163))
   (segment (start 79.121 57.912) (end 78.486 58.547) (width 0.2) (layer "B.Cu") (net 166))
   (segment (start 79.121 20.066) (end 79.121 57.912) (width 0.2) (layer "B.Cu") (net 166))
