File: Schematics/CPU/CPU.kicad_sch (KiCad schematic)
At the start: 69 parts, among them J1 3x32, J2 2x08, J3 2x08, J4 2x08, J5 2x01, J6 2x03, Q1 Q_NMOS_DGS, Q2 Q_NMOS_DGS, SW1 SW_DIP_x08, U1 68000D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

Commit message: a
Connections:
- net IS1: now also U7.11 (I1); no longer U7.12 (I2)
- net IS2: now also U7.12 (I2); no longer U7.13 (I3)
- net IS3: now also U7.13 (I3); no longer U7.3 (I6)
- net IS4: now also U7.1 (I4); no longer U7.11 (I1)
- net IS5: now also U7.2 (I5); no longer U7.1 (I4)
- net IS6: now also U7.3 (I6); no longer U7.2 (I5)
Changed lines of the file:
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@@
     (effects (font (size 1.27 1.27)) (justify left bottom))
+  )
+  (label "IS3" (at 271.653 318.389 180)
+    (effects (font (size 1.27 1.27)) (justify right bottom))
   )
   (label "IE6" (at 316.357 277.749 180)
@@
     (effects (font (size 1.27 1.27)) (justify right bottom))
   )
-  (label "IS3" (at 271.653 326.009 180)
-    (effects (font (size 1.27 1.27)) (justify right bottom))
-  )
-  (label "IS5" (at 271.653 320.929 180)
-    (effects (font (size 1.27 1.27)) (justify right bottom))
-  )
   (label "TMP16" (at 496.062 462.026 0)
     (effects (font (size 1.27 1.27)) (justify left bottom))
@@
     (effects (font (size 1.27 1.27)) (justify left bottom))
   )
+  (label "IS5" (at 271.653 323.469 180)
+    (effects (font (size 1.27 1.27)) (justify right bottom))
+  )
   (label "CLK_OSCI" (at 164.338 460.121 0)
     (effects (font (size 1.27 1.27)) (justify left bottom))
@@
     (effects (font (size 1.27 1.27)) (justify left bottom))
   )
+  (label "IS2" (at 271.653 315.849 180)
+    (effects (font (size 1.27 1.27)) (justify right bottom))
+  )
   (label "TMP19" (at 496.697 472.186 0)
     (effects (font (size 1.27 1.27)) (justify left bottom))
@@
     (effects (font (size 1.27 1.27)) (justify right bottom))
   )
+  (label "IS6" (at 271.653 326.009 180)
+    (effects (font (size 1.27 1.27)) (justify right bottom))
+  )
+  (label "IS4" (at 271.653 320.929 180)
+    (effects (font (size 1.27 1.27)) (justify right bottom))
+  )
   (label "~IACK1" (at 238.125 246.253 180)
     (effects (font (size 1.27 1.27)) (justify right bottom))
@@
     (effects (font (size 1.27 1.27)) (justify left bottom))
   )
-  (label "IS2" (at 271.653 318.389 180)
-    (effects (font (size 1.27 1.27)) (justify right bottom))
-  )
   (label "A21" (at 498.602 226.568 0)
     (effects (font (size 1.27 1.27)) (justify left bottom))
@@
     (effects (font (size 1.27 1.27)) (justify left bottom))
   )
-  (label "IS4" (at 271.653 313.309 180)
-    (effects (font (size 1.27 1.27)) (justify right bottom))
-  )
   (label "~RST" (at 466.725 172.085 0)
     (effects (font (size 1.27 1.27)) (justify left bottom))
@@
     (effects (font (size 1.27 1.27)) (justify right bottom))
   )
-  (label "IS6" (at 271.653 323.469 180)
-    (effects (font (size 1.27 1.27)) (justify right bottom))
-  )
   (label "~AS" (at 450.85 405.384 0)
     (effects (font (size 1.27 1.27)) (justify left bottom))
@@
     (effects (font (size 1.27 1.27)) (justify left bottom))
   )
-  (label "IS1" (at 271.653 315.849 180)
-    (effects (font (size 1.27 1.27)) (justify right bottom))
-  )
   (label "~BR" (at 466.725 167.005 0)
     (effects (font (size 1.27 1.27)) (justify left bottom))
@@
     (effects (font (size 1.27 1.27)) (justify left bottom))
   )
+  (label "IS1" (at 271.653 313.309 180)
+    (effects (font (size 1.27 1.27)) (justify right bottom))
+  )
   (label "~IACK1" (at 331.851 326.009 0)

Commit message: 7/18/2023
Connections:
- net GND: now also U15.10, U15.9, U8.3 (D0)
- net at U10.9 (~{PE}), U9.9 (~{PE}): now also U5.2; no longer U5.1
- net at U10.15 (TC), U11.10 (CET): now also U5.1; no longer U5.2
- no-connect marks 44 -> 46
Other:
- note added: "PLL only tested on breadboard PCB could be wrong and I don't know best C/R values Leave PLL chips unpopulated when not in use"
- moved on the sheet: U5A
