File: Schematics/MEMv1/MEM.kicad_sch (KiCad schematic)
At the start: 27 parts, among them J1 3x32, J2 Conn_02x04_Odd_Even, U1 SST39F040, U10 74HC245, U11 74HC245, U12 74LS85, U13 74LS138, U2 SST39F040, U3 AS6C4008-55PCN, U4 AS6C4008-55PCN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

Commit message: a
Parts:
- removed U12: 74LS85, Footpp:DIP-16, symbol 74xx:74LS85
- removed U13: 74LS138, Footpp:DIP-16, symbol 74xx:74LS138
Other:
- moved on the sheet: J1A
