File: Schematics/BP/BP.kicad_sch (KiCad schematic)
At the start: 23 parts, among them J1 3x32, J10 Conn_01x05_Male, J2 3x32, J3 3x32, J4 3x32, J5 3x32, J6 3x32, J7 3x32, J8 3x32, J9 Barrel_Jack_Switch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

Commit message: 7/18/2023
Parts:
- removed J10: Conn_01x05_Male, Connector_PinHeader_2.54mm:PinHeader_1x05_P2.54mm_Vertical, symbol Connector:Conn_01x05_Male
- added J10: 01x04, symbol Connector:Conn_01x04_Pin
Connections:
- net GND: now also J10.4 (Pin_4)
- net PWR_LED: now also J10.3 (Pin_3)
- net PWR_SWT_0: now also J10.1 (Pin_1)
- net PWR_SWT_1: now also J10.2 (Pin_2)
Other:
- moved on the sheet: C1, C2, C3, C4, C5, C6, C7, C8, C9, D1, D2, J1A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
