File: Schematics/IO/IO.kicad_sch (KiCad schematic)
At the start: 56 parts, among them J1 3x32, J10 1x03, J2 2x01, J3 2x01, J4 Conn_02x08_Top_Bottom, J5 Mini-DIN-6, J6 02x08, J7 Micro_SD_Card_Det, J8 2x01, J9 2x08, Q1 Q_NMOS_DGS, Q2 Q_NMOS_DGS, Q3 Q_NMOS_DGS, U1 74HC245, U10 74HC273, U11 74HC273, U12 74HC245, U13 74HC273, U14 74HC595, U15 74HC595, U16 DS1307+, U17 74LVC245, U18 LP2950-3.3_TO92, U2 74HC14, U3 74LS161, U4 74LS138, U5 74HC74, U6 74LS161, U7 74HC165, U8 74HC595, U9 74HC245, Y1 32768hz

Commit message: a
Connections:
- net SYS_PORT_SPI_CE0 is gone; now on net SPI_CE0: J9.6 (Pin_6)
Changed lines of the file:
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@@
     (effects (font (size 1.27 1.27)) (justify left bottom))
   )
-  (label "SYS_PORT_SPI_CE0" (at 211.836 375.412 180)
+  (label "SPI_CE0" (at 211.836 375.412 180)
     (effects (font (size 1.27 1.27)) (justify right bottom))
   )

Commit message: 7/18/2023
Parts:
- removed J10: 1x03, Connector_PinHeader_2.54mm:PinHeader_1x03_P2.54mm_Vertical, symbol Connector:Conn_01x03_Male
- added C19, C20, C21, C22, C23: 100n, Footpp:DIP-2_200_ELL, symbol Device:C
- added D2, D3: D, Diode_THT:D_DO-35_SOD27_P7.62mm_Horizontal, symbol Device:D
- added D4: LED, symbol Device:LED
- added R6: 220, Footpp:res, symbol Device:R
- added U19: 74HC157, symbol 74xx:74LS157
- C16: value C_Polarized -> C_Pol
- J4: value Conn_02x08_Top_Bottom -> Conn_02x08
- U3, U6: value 74LS161 -> 74HC161
- U4: value 74LS138 -> 74HC138
- U8: value 74HC595 -> 74HCT595
Connections:
- net +5V: now also C19.1, C20.1, C21.1, C22.1, C23.1, U19.16 (VCC)
- net CLK: now also U19.3 (I1a); no longer U3.2 (CP)
- net E: now also U3.2 (CP)
- net GND: now also U17.11 (B7), U17.12 (B6), U17.13 (B5), U17.14 (B4), U17.15 (B3), C19.2, C20.2, C21.2, C22.2, C23.2, D4.1 (K), U19.10 (I1c), U19.11 (I0c), U19.13 (I1d), U19.14 (I0d), U19.15 (E), U19.5 (I0b), U19.6 (I1b), U19.8 (GND)
- net ~DTACK: now also D2.1 (K), D3.1 (K)
- net at U5.3 (C), U6.2 (CP): now also U19.4 (Za)
- net at U5.2 (D), U5.9 (Q): now also D2.2 (A), R6.1
- net at U5.5 (Q), U6.7 (CEP): now also D3.2 (A)
- net <400KHZ: now reaches U3.13 (Q1)
- net <400KHZ: now also U19.2 (I0a)
- net CLK2: no longer names the net of U3.14 (Q0)
- net SD_DO renamed SPI_MISO
- net SYS_OUT_6: no longer names the net of J4.10 (Pin_10)
- net SYS_OUT_6: no longer U10.9 (Q3)
- new net: D4.2 (A), R6.2
- new net SPI_SPEED: U10.9 (Q3), U19.1 (S)
- no-connect marks 42 -> 46
Other:
- note added: "12.5pF <40Kohm ESR"
- note added: "GPIO"
- note added: "HDD BUSY LED"
- note added: "MUST BE HCT"
- note added: "MUST BE LVC"
- note removed: "CFS-20632768AZFB"
- note removed: "GEN IO"
- moved on the sheet: C1, C10, C11, C12, C13, C14, C15, C16, C17, C18, C2, C3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
